File: Transistor_AMPS/Two_transistor_AMP/Two_transistor_AMP.sch (KiCad schematic (older format))
At the start: 14 parts, among them J1 Conn_01x02, J2 Conn_01x02, Q1 BC546, Q2 BC546

Commit message: Majasdarbs update
Parts:
- removed J1, J2: Conn_01x02, TerminalBlock:TerminalBlock_bornier-2_P5.08mm, symbol Connector_Generic:Conn_01x02
- removed Q1, Q2: BC546, Package_TO_SOT_THT:TO-92L_Inline, symbol Device:Q_NPN_BCE
- added J1, J2, J3: Screw_Terminal_01x02, TerminalBlock:TerminalBlock_bornier-2_P5.08mm, symbol Connector:Screw_Terminal_01x02
- added Q1, Q2: BC546, Package_TO_SOT_THT:TO-92L_Inline, symbol Device:Q_NPN_CBE
Connections:
- net +9V: now also J2.2 (Pin_2), Q2.1 (C)
- net GNDREF: now also J1.1 (Pin_1), J2.1 (Pin_1), J3.2 (Pin_2)
- net at C1.1, R1.2, R2.1: now also Q1.2 (B)
- net at C5.2, R5.1: now also Q2.3 (E)
- net at C3.2, R3.2: now also Q1.1 (C)
- net at C2.1, R4.1: now also Q1.3 (E)
- net at C3.1: now also Q2.2 (B)
- net at C5.1: now also J3.1 (Pin_1)
- net at C1.2: now also J1.2 (Pin_2)
Changed lines of the file:
@@
-$EndComp
-$Comp
-L Device:Q_NPN_BCE Q1
-U 1 1 61803CD7
-P 6350 2600
-F 0 "Q1" H 6541 2646 50  0000 L CNN
-F 1 "BC546" H 6541 2555 50  0000 L CNN
-F 2 "Package_TO_SOT_THT:TO-92L_Inline" H 6550 2700 50  0001 C CNN
-F 3 "~" H 6350 2600 50  0001 C CNN
-	1    6350 2600
-	1    0    0    -1
-$EndComp
-$Comp
-L Device:Q_NPN_BCE Q2
-U 1 1 61804A5F
-P 7650 2600
-F 0 "Q2" H 7841 2646 50  0000 L CNN
-F 1 "BC546" H 7841 2555 50  0000 L CNN
-F 2 "Package_TO_SOT_THT:TO-92L_Inline" H 7850 2700 50  0001 C CNN
-F 3 "~" H 7650 2600 50  0001 C CNN
-	1    7650 2600
-	1    0    0    -1
 $EndComp
 $Comp
@@
 Wire Wire Line
 	5900 2600 5750 2600
-$Comp
-L Connector_Generic:Conn_01x02 J2
-U 1 1 618286F2
+Wire Wire Line
+	8250 2900 8350 2900
+Wire Wire Line
+	8350 3000 8350 3200
+Wire Wire Line
+	8350 3200 7750 3200
+Connection ~ 7750 3200
+Wire Wire Line
+	5450 2600 5550 2600
+Wire Wire Line
+	5450 2700 5450 3200
+Wire Wire Line
+	5450 3200 5900 3200
+Connection ~ 5900 3200
+$Comp
+L Connector:Screw_Terminal_01x02 J2
+U 1 1 61A11392
+P 8550 2350
+F 0 "J2" H 8630 2342 50  0000 L CNN
+F 1 "Screw_Terminal_01x02" H 8630 2251 50  0000 L CNN
+F 2 "TerminalBlock:TerminalBlock_bornier-2_P5.08mm" H 8550 2350 50  0001 C CNN
+F 3 "~" H 8550 2350 50  0001 C CNN
+	1    8550 2350
+	1    0    0    -1
+$EndComp
+$Comp
+L Connector:Screw_Terminal_01x02 J3
+U 1 1 61A1219C
 P 8550 2900
-F 0 "J2" H 8630 2846 50  0000 L CNN
-F 1 "Conn_01x02" H 8630 2801 50  0001 L CNN
+F 0 "J3" H 8630 2892 50  0000 L CNN
+F 1 "Screw_Terminal_01x02" H 8630 2801 50  0000 L CNN
 F 2 "TerminalBlock:TerminalBlock_bornier-2_P5.08mm" H 8550 2900 50  0001 C CNN
 F 3 "~" H 8550 2900 50  0001 C CNN
@@
 $EndComp
 $Comp
-L Connector_Generic:Conn_01x02 J1
-U 1 1 61829940
+L Connector:Screw_Terminal_01x02 J1
+U 1 1 61A12F31
 P 5250 2700
-F 0 "J1" H 5400 2650 50  0000 C CNN
-F 1 "Conn_01x02" H 5330 2601 50  0001 L CNN
+F 0 "J1" H 5168 2375 50  0000 C CNN
+F 1 "Screw_Terminal_01x02" H 5168 2466 50  0000 C CNN
 F 2 "TerminalBlock:TerminalBlock_bornier-2_P5.08mm" H 5250 2700 50  0001 C CNN
 F 3 "~" H 5250 2700 50  0001 C CNN
@@
 	-1   0    0    1
 $EndComp
-Wire Wire Line
-	8250 2900 8350 2900
-Wire Wire Line
-	8350 3000 8350 3200
-Wire Wire Line
-	8350 3200 7750 3200
-Connection ~ 7750 3200
-Wire Wire Line
-	5450 2600 5550 2600
-Wire Wire Line
-	5450 2700 5450 3200
-Wire Wire Line
-	5450 3200 5900 3200
-Connection ~ 5900 3200
+$Comp
+L Device:Q_NPN_CBE Q2
+U 1 1 61A185CC
+P 7650 2600
+F 0 "Q2" H 7841 2646 50  0000 L CNN
+F 1 "BC546" H 7841 2555 50  0000 L CNN
+F 2 "Package_TO_SOT_THT:TO-92L_Inline" H 7850 2700 50  0001 C CNN
+F 3 "~" H 7650 2600 50  0001 C CNN
+	1    7650 2600
+	1    0    0    -1
+$EndComp
+$Comp
+L Device:Q_NPN_CBE Q1
+U 1 1 61A190D5
+P 6350 2600
+F 0 "Q1" H 6541 2646 50  0000 L CNN
+F 1 "BC546" H 6541 2555 50  0000 L CNN
+F 2 "Package_TO_SOT_THT:TO-92L_Inline" H 6550 2700 50  0001 C CNN
+F 3 "~" H 6350 2600 50  0001 C CNN
+	1    6350 2600
+	1    0    0    -1
+$EndComp
+$Comp
+L power:+9V #PWR01
+U 1 1 61A13F4D
+P 8350 2450
+F 0 "#PWR01" H 8350 2300 50  0001 C CNN
+F 1 "+9V" H 8365 2623 50  0000 C CNN
+F 2 "" H 8350 2450 50  0001 C CNN
+F 3 "" H 8350 2450 50  0001 C CNN
+	1    8350 2450
+	-1   0    0    1
+$EndComp
+$Comp
+L power:GNDREF #PWR02
+U 1 1 61A1370D
+P 8350 2350
+F 0 "#PWR02" H 8350 2100 50  0001 C CNN
+F 1 "GNDREF" H 8355 2177 50  0000 C CNN
+F 2 "" H 8350 2350 50  0001 C CNN
+F 3 "" H 8350 2350 50  0001 C CNN
+	1    8350 2350
+	-1   0    0    1
+$EndComp
 $EndSCHEMATC
