File: Transistor_AMPS/Two_transistor_AMP/Two_transistor_AMP.kicad_pcb (KiCad board)
At the start: 2 copper layers, 58.7 x 34 mm, 15 parts, among them Q1 BC546, Q2 BC546

Commit message: majasdarbs
Routing:
- net +9V: track 0.00 -> 47.1 mm
- net Net-(C1-Pad1): track 0.00 -> 24.3 mm
- net Net-(C2-Pad1): track 0.00 -> 19.1 mm
- net Net-(C3-Pad2): track 0.00 -> 18.2 mm
- net Net-(C5-Pad2): track 0.00 -> 15.6 mm
- net Net-(C1-Pad2): track 0.00 -> 14.9 mm
- net Net-(C3-Pad1): track 0.00 -> 6.67 mm
- net Net-(C5-Pad1): track 0.00 -> 6.47 mm
- added copper zone on B.Cu, net GNDREF
- added copper zone on F.Cu, net GNDREF
